File: ab18x5-breakout/ab18x5-breakout.kicad_pcb (KiCad board)
At the start: 2 copper layers, 18.3 x 15.7 mm, 6 parts, among them J1 CONN_01X07, J2 CONN_01X07, U1 AB1815, Y1 Crystal

Commit message: adding 3D models and better silk screen
Parts:
- added G***: LOGO, ab18x5-breakout:oshw, F.Cu at (216.9, 159.8)
Other:
- board text added: "1 nRST"
- board text added: "2 WDI"
- board text added: "3 nEXTR"
- board text added: "4 nIRQ2"
- board text added: "5 VBAT"
- board text added: "6 SDO"
- board text added: "7 SCL"
- board text added: "EXTI 10"
- board text added: "SDI 9"
- board text added: "VCC 13"
- board text added: "VSS PAD"
- board text added: "frank-buss.de"
- board text added: "nCE 12"
- board text added: "nIRQ 11"
- board text added: "nIRQ3 8"
- board text removed: "EXTI"
- board text removed: "SCL"
- board text removed: "SDI"
- board text removed: "SDO"
- board text removed: "VBAT"
- board text removed: "VCC"
- board text removed: "VSS"
- board text removed: "WDI"
- board text removed: "nCE"
- board text removed: "nEXTR"
- board text removed: "nIRQ"
- board text removed: "nIRQ2"
- board text removed: "nIRQ3"
- board text removed: "nRST"
